File: pcb/stomp_00/digitalinput.kicad_sch (KiCad schematic)
At the start: 1 part, among them U11 74HC165

Commit message: adding all the components...
Parts:
- added SW1: SW_DIP_x04, symbol Switch:SW_DIP_x04
- added U13: 74HC165, symbol 74xx:74HC165
Changed lines of the file:
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@@
 (kicad_sch (version 20230121) (generator eeschema)
   (paper "A4")
+  (text_box "16 digital inputs. Footswitches, tactile buttons, toggle switches. Allow DIP switch on PCB. Need to think about whether to add pullups to all inputs."
+    (at 109.22 33.02 0) (size 52.07 21.59)
+    (stroke (width 0) (type default))
+    (fill (type none))
+    (effects (font (size 1.27 1.27)) (justify left top))
+  )
+  (symbol (lib_id "Switch:SW_DIP_x04") (at 111.76 165.1 0) (unit 1)
+    (in_bom yes) (on_board yes) (dnp no) (fields_autoplaced)
+    (property "Reference" "SW1" (at 111.76 153.67 0)
+      (effects (font (size 1.27 1.27)))
+    )
+    (property "Value" "SW_DIP_x04" (at 111.76 156.21 0)
+      (effects (font (size 1.27 1.27)))
+    )
+    (property "Footprint" "" (at 111.76 165.1 0)
+      (effects (font (size 1.27 1.27)) hide)
+    )
+    (property "Datasheet" "~" (at 111.76 165.1 0)
+      (effects (font (size 1.27 1.27)) hide)
+    )
+    (pin "1")
+    (pin "2")
+    (pin "3")
+    (pin "4")
+    (pin "5")
+    (pin "6")
+    (pin "7")
+    (pin "8")
+    (instances
+      (project "stomp_00"
+        (path "/8f4a2eb0-078b-46cb-b534-a4acd11d130e/c212ffd9-4be4-4b31-b430-fe718bd94dd5"
+          (reference "SW1") (unit 1)
+        )
+      )
+    )
+  )
+  (symbol (lib_id "74xx:74HC165") (at 142.24 153.67 0) (unit 1)
+    (in_bom yes) (on_board yes) (dnp no) (fields_autoplaced)
+    (property "Reference" "U13" (at 144.1959 132.08 0)
+      (effects (font (size 1.27 1.27)) (justify left))
+    )
+    (property "Value" "74HC165" (at 144.1959 134.62 0)
+      (effects (font (size 1.27 1.27)) (justify left))
+    )
+    (property "Footprint" "" (at 142.24 153.67 0)
+      (effects (font (size 1.27 1.27)) hide)
+    )
+    (property "Datasheet" "https://assets.nexperia.com/documents/data-sheet/74HC_HCT165.pdf" (at 142.24 153.67 0)
+      (effects (font (size 1.27 1.27)) hide)
+    )
+    (pin "1")
+    (pin "10")
+    (pin "11")
+    (pin "12")
+    (pin "13")
+    (pin "14")
+    (pin "15")
+    (pin "16")
+    (pin "2")
+    (pin "3")
+    (pin "4")
+    (pin "5")
+    (pin "6")
+    (pin "7")
+    (pin "8")
+    (pin "9")
+    (instances
+      (project "stomp_00"
+        (path "/8f4a2eb0-078b-46cb-b534-a4acd11d130e/c212ffd9-4be4-4b31-b430-fe718bd94dd5"
+          (reference "U13") (unit 1)
+        )
+        (path "/8f4a2eb0-078b-46cb-b534-a4acd11d130e/3c05a139-0458-42fa-b53c-1db5d985c9e4"
+          (reference "U12") (unit 1)
+        )
+      )
+    )
+  )
   (symbol (lib_id "74xx:74HC165") (at 142.24 95.25 0) (unit 1)
     (in_bom yes) (on_board yes) (dnp no) (fields_autoplaced)

Commit message: taking shape...
Parts:
- SW1: footprint (none) -> Button_Switch_THT:SW_DIP_SPSTx04_Slide_9.78x12.34mm_W7.62mm_P2.54mm
- U11, U13: footprint (none) -> Package_SO:SOIC-16_3.9x9.9mm_P1.27mm
Changed lines of the file:
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@@
       (effects (font (size 1.27 1.27)))
     )
-    (property "Footprint" "" (at 111.76 165.1 0)
+    (property "Footprint" "Button_Switch_THT:SW_DIP_SPSTx04_Slide_9.78x12.34mm_W7.62mm_P2.54mm" (at 111.76 165.1 0)
       (effects (font (size 1.27 1.27)) hide)
     )
@@
       (effects (font (size 1.27 1.27)) (justify left))
     )
-    (property "Footprint" "" (at 142.24 153.67 0)
+    (property "Footprint" "Package_SO:SOIC-16_3.9x9.9mm_P1.27mm" (at 142.24 153.67 0)
       (effects (font (size 1.27 1.27)) hide)
     )
@@
       (effects (font (size 1.27 1.27)) (justify left))
     )
-    (property "Footprint" "" (at 142.24 95.25 0)
+    (property "Footprint" "Package_SO:SOIC-16_3.9x9.9mm_P1.27mm" (at 142.24 95.25 0)
       (effects (font (size 1.27 1.27)) hide)
     )
