File: pcb/stomp_00/digitaloutput.kicad_sch (KiCad schematic)
At the start: 9 parts, among them U12 74HC595

Commit message: adding all the components...
Changed lines of the file:
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@@
 (kicad_sch (version 20230121) (generator eeschema)
   (paper "A4")
+  (text_box "Digital outputs. Mainly for LEDs. Resistors?"
+    (at 101.6 24.13 0) (size 58.42 26.67)
+    (stroke (width 0) (type default))
+    (fill (type none))
+    (effects (font (size 1.27 1.27)) (justify left top))
+  )
   (symbol (lib_id "Device:R_US") (at 189.23 104.14 0) (unit 1)
     (in_bom yes) (on_board yes) (dnp no) (fields_autoplaced)
@@
         (path "/8f4a2eb0-078b-46cb-b534-a4acd11d130e/3c05a139-0458-42fa-b53c-1db5d985c9e4"
           (reference "R8") (unit 1)
+        )
+        (path "/8f4a2eb0-078b-46cb-b534-a4acd11d130e/178dbe3d-cc28-49ed-9d60-e09a02802844"
+          (reference "R19") (unit 1)
         )
       )
@@
           (reference "U12") (unit 1)
         )
+        (path "/8f4a2eb0-078b-46cb-b534-a4acd11d130e/178dbe3d-cc28-49ed-9d60-e09a02802844"
+          (reference "U14") (unit 1)
+        )
       )
     )
@@
           (reference "R9") (unit 1)
         )
+        (path "/8f4a2eb0-078b-46cb-b534-a4acd11d130e/178dbe3d-cc28-49ed-9d60-e09a02802844"
+          (reference "R20") (unit 1)
+        )
       )
     )
@@
           (reference "R4") (unit 1)
         )
+        (path "/8f4a2eb0-078b-46cb-b534-a4acd11d130e/178dbe3d-cc28-49ed-9d60-e09a02802844"
+          (reference "R17") (unit 1)
+        )
       )
     )
@@
           (reference "R10") (unit 1)
         )
+        (path "/8f4a2eb0-078b-46cb-b534-a4acd11d130e/178dbe3d-cc28-49ed-9d60-e09a02802844"
+          (reference "R23") (unit 1)
+        )
       )
     )
@@
           (reference "R11") (unit 1)
         )
+        (path "/8f4a2eb0-078b-46cb-b534-a4acd11d130e/178dbe3d-cc28-49ed-9d60-e09a02802844"
+          (reference "R24") (unit 1)
+        )
       )
     )
@@
           (reference "R7") (unit 1)
         )
+        (path "/8f4a2eb0-078b-46cb-b534-a4acd11d130e/178dbe3d-cc28-49ed-9d60-e09a02802844"
+          (reference "R22") (unit 1)
+        )
       )
     )
@@
           (reference "R6") (unit 1)
         )
+        (path "/8f4a2eb0-078b-46cb-b534-a4acd11d130e/178dbe3d-cc28-49ed-9d60-e09a02802844"
+          (reference "R18") (unit 1)
+        )
       )
     )
@@
           (reference "R5") (unit 1)
         )
-      )
+        (path "/8f4a2eb0-078b-46cb-b534-a4acd11d130e/178dbe3d-cc28-49ed-9d60-e09a02802844"
+          (reference "R21") (unit 1)
+        )
+      )

Commit message: taking shape...
Parts:
- R10, R11, R4, R5, R6, R7, R8, R9: footprint (none) -> Resistor_SMD:R_0603_1608Metric
- U12: footprint (none) -> Package_SO:SOIC-16_3.9x9.9mm_P1.27mm
Changed lines of the file:
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@@
       (effects (font (size 1.27 1.27)) (justify left))
     )
-    (property "Footprint" "" (at 190.246 104.394 90)
+    (property "Footprint" "Resistor_SMD:R_0603_1608Metric" (at 190.246 104.394 90)
       (effects (font (size 1.27 1.27)) hide)
     )
@@
       (effects (font (size 1.27 1.27)) (justify left))
     )
-    (property "Footprint" "" (at 144.78 95.25 0)
+    (property "Footprint" "Package_SO:SOIC-16_3.9x9.9mm_P1.27mm" (at 144.78 95.25 0)
       (effects (font (size 1.27 1.27)) hide)
     )
@@
       (effects (font (size 1.27 1.27)) (justify left))
     )
-    (property "Footprint" "" (at 190.246 118.364 90)
+    (property "Footprint" "Resistor_SMD:R_0603_1608Metric" (at 190.246 118.364 90)
       (effects (font (size 1.27 1.27)) hide)
     )
@@
       (effects (font (size 1.27 1.27)) (justify left))
     )
-    (property "Footprint" "" (at 190.246 76.454 90)
+    (property "Footprint" "Resistor_SMD:R_0603_1608Metric" (at 190.246 76.454 90)
       (effects (font (size 1.27 1.27)) hide)
     )
@@
       (effects (font (size 1.27 1.27)) (justify left))
     )
-    (property "Footprint" "" (at 202.946 104.394 90)
+    (property "Footprint" "Resistor_SMD:R_0603_1608Metric" (at 202.946 104.394 90)
       (effects (font (size 1.27 1.27)) hide)
     )
@@
       (effects (font (size 1.27 1.27)) (justify left))
     )
-    (property "Footprint" "" (at 202.946 118.364 90)
+    (property "Footprint" "Resistor_SMD:R_0603_1608Metric" (at 202.946 118.364 90)
       (effects (font (size 1.27 1.27)) hide)
     )
@@
       (effects (font (size 1.27 1.27)) (justify left))
     )
-    (property "Footprint" "" (at 202.946 90.424 90)
+    (property "Footprint" "Resistor_SMD:R_0603_1608Metric" (at 202.946 90.424 90)
       (effects (font (size 1.27 1.27)) hide)
     )
@@
       (effects (font (size 1.27 1.27)) (justify left))
     )
-    (property "Footprint" "" (at 190.246 90.424 90)
+    (property "Footprint" "Resistor_SMD:R_0603_1608Metric" (at 190.246 90.424 90)
       (effects (font (size 1.27 1.27)) hide)
     )
@@
       (effects (font (size 1.27 1.27)) (justify left))
     )
-    (property "Footprint" "" (at 202.946 76.454 90)
-      (effects (font (size 1.27 1.27)) hide)
-    )
+    (property "Footprint" "Resistor_SMD:R_0603_1608Metric" (at 202.946 76.454 90)
+      (effects (font (size 1.27 1.27)) hide)
+    )
