File: pcb/stomp_00/midi.kicad_sch (KiCad schematic)
At the start: 10 parts, among them J10 AudioJack3, J11 AudioJack3, U13 6N138

Commit message: taking shape...
Parts:
- J10, J11: footprint (none) -> Connector_PinHeader_2.54mm:PinHeader_1x03_P2.54mm_Vertical
- R17, R18, R19, R20, R21: footprint (none) -> Resistor_SMD:R_0603_1608Metric
Changed lines of the file:
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@@
       (effects (font (size 1.27 1.27)))
     )
-    (property "Footprint" "" (at 208.28 147.32 0)
+    (property "Footprint" "Connector_PinHeader_2.54mm:PinHeader_1x03_P2.54mm_Vertical" (at 208.28 147.32 0)
       (effects (font (size 1.27 1.27)) hide)
     )
@@
       (effects (font (size 1.27 1.27)) (justify left))
     )
-    (property "Footprint" "" (at 77.216 136.144 90)
+    (property "Footprint" "Resistor_SMD:R_0603_1608Metric" (at 77.216 136.144 90)
       (effects (font (size 1.27 1.27)) hide)
     )
@@
       (effects (font (size 1.27 1.27)) (justify left))
     )
-    (property "Footprint" "" (at 185.166 138.684 90)
+    (property "Footprint" "Resistor_SMD:R_0603_1608Metric" (at 185.166 138.684 90)
       (effects (font (size 1.27 1.27)) hide)
     )
@@
       (effects (font (size 1.27 1.27)) (justify left))
     )
-    (property "Footprint" "" (at 103.886 138.684 90)
+    (property "Footprint" "Resistor_SMD:R_0603_1608Metric" (at 103.886 138.684 90)
       (effects (font (size 1.27 1.27)) hide)
     )
@@
       (effects (font (size 1.27 1.27)) (justify left))
     )
-    (property "Footprint" "" (at 100.076 153.924 90)
+    (property "Footprint" "Resistor_SMD:R_0603_1608Metric" (at 100.076 153.924 90)
       (effects (font (size 1.27 1.27)) hide)
     )
@@
       (effects (font (size 1.27 1.27)) (justify left))
     )
-    (property "Footprint" "" (at 173.736 150.114 90)
+    (property "Footprint" "Resistor_SMD:R_0603_1608Metric" (at 173.736 150.114 90)
       (effects (font (size 1.27 1.27)) hide)
     )
@@
       (effects (font (size 1.27 1.27)))
     )
-    (property "Footprint" "" (at 60.96 148.59 0)
-      (effects (font (size 1.27 1.27)) hide)
-    )
+    (property "Footprint" "Connector_PinHeader_2.54mm:PinHeader_1x03_P2.54mm_Vertical" (at 60.96 148.59 0)
+      (effects (font (size 1.27 1.27)) hide)
+    )
