File: pcb/stomp_00/stomp_00.kicad_pcb (KiCad board)
At the start: 2 copper layers, 54 x 106 mm, 88 parts, among them J1 Headphones, J10 Conn_01x18_Pin, J11 Conn_01x18_Pin, J12 Conn_01x18_Pin, J13 Conn_01x18_Pin, J14 Conn_01x18_Pin, J15 Conn_01x18_Pin, J16 Conn_01x18_Pin, J17 Conn_01x18_Pin, J18 Conn_01x18_Pin, J2 Footswitch_breakout, J3 GuitarInput1, J5 GuitarOutput1, J6 Conn_02x05_Counter_Clockwise, J8 Barrel_Jack, J9 Conn_01x18_Pin, SW2 Footswitch, U1 AP7313-18SAG, U2 TL072, U3 SGTL5000XNLA3, U7 Teensy4.1, U8 TPS54331DR

Commit message: not much
Parts:
- moved C18 104.9 mm to (34.3, 20.0)
- moved C19 99.3 mm to (34.3, 28.5)
- moved C20 99.3 mm to (34.3, 31.0)
- moved C21 97.8 mm to (37.5, 23.8), turned to 90 degrees
- moved C23 96.9 mm to (38.3, 34.5)
- moved C26 96.9 mm to (42.3, 29.5)
- moved C22 96.9 mm to (42.3, 32.0)
- moved C24 96.9 mm to (42.3, 24.5)
- moved C25 96.9 mm to (42.3, 27.0)
- moved R19 88.9 mm to (38.3, 45.0)
- moved R20 88.9 mm to (42.3, 35.0)
- moved R21 88.9 mm to (42.3, 37.5)
- moved R22 88.9 mm to (42.3, 40.0)
- moved R16 34.7 mm to (34.3, 38.5)
- moved R17 34.7 mm to (34.3, 36.0)
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- renumbered C23 to C1, C14 to C10, C10 to C11, C15 to C12, C18 to C13, C12 to C14, C16 to C15, C11 to C16, C2 to C18, C3 to C19, C28 to C2, C4 to C20, C1 to C21, C25 to C22, C5 to C23, C9 to C24, C21 to C25, C22 to C26, C27 to C3, C26 to C4, C31 to C5, C24 to C6, C8 to C7, C13 to C8, C7 to C9, D6 to D1, D1 to D2, D4 to D3, D5 to D4, J9 to J1, J18 to J10, J8 to J11, J1 to J12, J2 to J13, J6 to J14, J3 to J15, J5 to J16, J10 to J2, J11 to J3, J12 to J4, J13 to J5, J14 to J6, J15 to J7, J16 to J8, J17 to J9, L2 to L1, R27 to R1, R5 to R10, R13 to R11, R8 to R12, R14 to R13, R9 to R14, R2 to R16, R1 to R17, R3 to R18, R17 to R19, R25 to R2, R18 to R20, R19 to R21, R20 to R22, R16 to R23, R26 to R3, R10 to R5, R11 to R8, R12 to R9, SW2 to SW1, U7 to U1, U8 to U2, U2 to U3, U1 to U4, U3 to U5

Commit message: layout getting closer
Parts:
- removed J14: Conn_02x05_Counter_Clockwise, Connector_PinHeader_2.54mm:PinHeader_2x05_P2.54mm_Vertical
- added JP1: Jumper_2_Bridged, Jumper:SolderJumper-2_P1.3mm_Bridged2Bar_RoundedPad1.0x1.5mm, F.Cu at (36.2, 48.5)
- added JP2: Jumper_2_Bridged, Jumper:SolderJumper-2_P1.3mm_Bridged2Bar_RoundedPad1.0x1.5mm, F.Cu at (36.6, 37.5)
- added R12: Gain, Resistor_THT:R_Axial_DIN0207_L6.3mm_D2.5mm_P7.62mm_Horizontal, F.Cu at (41.8, 51.8)
- added R14: Gain, Resistor_THT:R_Axial_DIN0207_L6.3mm_D2.5mm_P7.62mm_Horizontal, F.Cu at (34.7, 34.3)
- R13: renamed from R12; value 4.2k -> 4.7k
- R15: renamed from R13; value 4.2k -> 4.7k
- moved R4 101.7 mm to (45.1, 90.8)
- moved C17 98.7 mm to (37.5, 28.1), turned to 90 degrees
- moved C16 98.0 mm to (35.9, 28.1), turned to 90 degrees
- moved C14 98.0 mm to (34.3, 31.2), turned to -90 degrees
- moved R5 97.3 mm to (48.2, 90.8)
- moved R9 96.1 mm to (48.2, 87.6)
- moved R7 94.9 mm to (48.2, 86.0)
- moved R6 94.4 mm to (45.1, 86.0)
- moved C15 93.0 mm to (39.1, 31.2), turned to 90 degrees
- moved R8 91.0 mm to (45.1, 87.6)
- moved C13 88.5 mm to (34.8, 42.6), turned to 90 degrees
- moved C12 85.1 mm to (39.6, 36.8)
- moved C10 76.7 mm to (42.0, 42.3), turned to 90 degrees
- moved C11 74.5 mm to (39.1, 49.3), turned to 180 degrees
- moved C9 72.5 mm to (42.0, 45.4), turned to -90 degrees
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- renumbered JP8 to JP10, JP9 to JP11, JP1 to JP3, JP2 to JP4, JP3 to JP5, JP4 to JP6, JP5 to JP7, JP6 to JP8, JP7 to JP9, R14 to R16, R15 to R17, R16 to R18, R17 to R19, R18 to R20, R19 to R21, R20 to R22, R21 to R23, R22 to R24, R23 to R25
Connections:
- C11 pad 2: Net-(C11-Pad2) -> Net-(JP1-B)
- C12 pad 2: Net-(C12-Pad2) -> Net-(JP2-B)
- C7 pad 1: INSTRUMENT_IN_L -> PREAMP_IN_L
- C8 pad 1: INSTRUMENT_IN_R -> PREAMP_IN_R
- J1 pad 1: +3.3V -> +9V
- J1 pad 10: unconnected-(J1-Pin_10-Pad10) -> LINE_IN_L
- J1 pad 11: unconnected-(J1-Pin_11-Pad11) -> LINE_IN_R
- J1 pad 12: unconnected-(J1-Pin_12-Pad12) -> LINE_OUT_L
- J1 pad 13: unconnected-(J1-Pin_13-Pad13) -> LINE_OUT_R
- J1 pad 14: unconnected-(J1-Pin_14-Pad14) -> LED_NEG
- J1 pad 15: unconnected-(J1-Pin_15-Pad15) -> GND
- J1 pad 2: +3.3V -> +9V
- J1 pad 4: unconnected-(J1-Pin_4-Pad4) -> +3.3V
- J1 pad 5: unconnected-(J1-Pin_5-Pad5) -> +3.3V
- J1 pad 6: unconnected-(J1-Pin_6-Pad6) -> JACK_IN
- J1 pad 7: unconnected-(J1-Pin_7-Pad7) -> JACK_OUT
- J1 pad 8: unconnected-(J1-Pin_8-Pad8) -> PREAMP_IN_L
- J1 pad 9: unconnected-(J1-Pin_9-Pad9) -> PREAMP_IN_R
- JP11 pad 1: INSTRUMENT_IN_L -> PREAMP_IN_L
- JP5 pad 2: INSTRUMENT_IN_L -> PREAMP_IN_L
- R13 pad 2: Net-(C11-Pad2) -> Net-(JP1-A)
- R15 pad 2: Net-(C12-Pad2) -> Net-(JP2-A)
- R16 pad 1: Net-(C11-Pad2) -> Net-(JP1-B)
- R17 pad 1: Net-(C12-Pad2) -> Net-(JP2-B)
- R4 pad 1: INSTRUMENT_IN_L -> PREAMP_IN_L
- R5 pad 1: INSTRUMENT_IN_R -> PREAMP_IN_R
- U3 pad 1: Net-(C11-Pad2) -> Net-(JP1-B)
- U3 pad 7: Net-(C12-Pad2) -> Net-(JP2-B)
Other:
- board text added: "9V"
- board text removed: "pedal in dac inL dac inR led neg gnd"
- board text removed: "pedal out dac outL dac outR h/p L h/p R"
