File: pcb/stomp_00/stomp_00.kicad_pcb (KiCad board)
At the start: 2 copper layers, 54 x 106 mm, 91 parts, among them J1 Conn_01x18_Pin, J10 Conn_01x18_Pin, J11 Barrel_Jack, J12 Headphones, J13 Footswitch_breakout, J15 GuitarInput1, J16 GuitarOutput1, J2 Conn_01x18_Pin, J3 Conn_01x18_Pin, J4 Conn_01x18_Pin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

Commit message: not much
Parts:
- moved JP3 8.77 mm to (10.0, 76.8), turned to -90 degrees
- moved JP6 8.66 mm to (12.6, 73.3), turned to -90 degrees
- moved JP7 7.12 mm to (12.6, 70.0)
- moved JP8 5.73 mm to (15.2, 76.8)
- moved JP10 4.47 mm to (15.2, 70.0)
- moved JP4 4.24 mm to (10.0, 73.3)
- moved JP9 2.42 mm to (15.2, 73.3)
- moved JP5 0.40 mm to (10.0, 70.0)
Changed lines of the file:
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@@
   )
   (footprint "Jumper:SolderJumper-2_P1.3mm_Bridged2Bar_RoundedPad1.0x1.5mm" (layer "B.Cu")
-    (at 4 74.35 90)
+    (at 12.6 73.35 -90)
     (descr "SMD Solder Jumper, 1x1.5mm, rounded Pads, 0.3mm gap, bridged with 2 copper strips")
     (tags "net tie solder jumper bridged")
@@
     (fp_line (start 1.65 -1.25) (end 1.65 1.25)
       (stroke (width 0.05) (type solid)) (layer "B.CrtYd"))
-    (pad "1" smd custom (at -0.65 0 90) (size 1 0.5) (layers "B.Cu" "B.Mask")
+    (pad "1" smd custom (at -0.65 0 270) (size 1 0.5) (layers "B.Cu" "B.Mask")
       (net 62 "FOOTSWITCH_5") (pinfunction "A") (pintype "passive") (zone_connect 2) (thermal_bridge_angle 45)
       (options (clearance outline) (anchor rect))
@@
           (width 0) (fill yes))
       ))
-    (pad "2" smd custom (at 0.65 0 90) (size 1 0.5) (layers "B.Cu" "B.Mask")
+    (pad "2" smd custom (at 0.65 0 270) (size 1 0.5) (layers "B.Cu" "B.Mask")
       (net 9 "GNDA") (pinfunction "B") (pintype "passive") (zone_connect 2) (thermal_bridge_angle 45)
       (options (clearance outline) (anchor rect))
@@
   )
   (footprint "Jumper:SolderJumper-2_P1.3mm_Bridged2Bar_RoundedPad1.0x1.5mm" (layer "B.Cu")
-    (at 7 74.35 -90)
+    (at 12.6 69.95 -90)
     (descr "SMD Solder Jumper, 1x1.5mm, rounded Pads, 0.3mm gap, bridged with 2 copper strips")
     (tags "net tie solder jumper bridged")
@@
   )
   (footprint "Jumper:SolderJumper-2_P1.3mm_Bridged2Bar_RoundedPad1.0x1.5mm" (layer "B.Cu")
-    (at 13 74.35 90)
+    (at 15.2 73.35 90)
     (descr "SMD Solder Jumper, 1x1.5mm, rounded Pads, 0.3mm gap, bridged with 2 copper strips")
     (tags "net tie solder jumper bridged")
@@
   )
   (footprint "Jumper:SolderJumper-2_P1.3mm_Bridged2Bar_RoundedPad1.0x1.5mm" (layer "B.Cu")
-    (at 16 74.35 90)
+    (at 15.2 69.95 90)
     (descr "SMD Solder Jumper, 1x1.5mm, rounded Pads, 0.3mm gap, bridged with 2 copper strips")
     (tags "net tie solder jumper bridged")
@@
   )
   (footprint "Jumper:SolderJumper-2_P1.3mm_Bridged2Bar_RoundedPad1.0x1.5mm" (layer "B.Cu")
-    (at 10 70.35 -90)
+    (at 10 69.95 -90)
     (descr "SMD Solder Jumper, 1x1.5mm, rounded Pads, 0.3mm gap, bridged with 2 copper strips")
     (tags "net tie solder jumper bridged")
@@
   )
   (footprint "Jumper:SolderJumper-2_P1.3mm_Bridged2Bar_RoundedPad1.0x1.5mm" (layer "B.Cu")
-    (at 10 74.35 90)
+    (at 15.2 76.75 90)
     (descr "SMD Solder Jumper, 1x1.5mm, rounded Pads, 0.3mm gap, bridged with 2 copper strips")
     (tags "net tie solder jumper bridged")
@@
   )
   (footprint "Jumper:SolderJumper-2_P1.3mm_Bridged2Bar_RoundedPad1.0x1.5mm" (layer "B.Cu")
-    (at 4 70.35 90)
+    (at 10 76.75 -90)
     (descr "SMD Solder Jumper, 1x1.5mm, rounded Pads, 0.3mm gap, bridged with 2 copper strips")
     (tags "net tie solder jumper bridged")
@@
     (fp_line (start 1.65 -1.25) (end 1.65 1.25)
       (stroke (width 0.05) (type solid)) (layer "B.CrtYd"))
-    (pad "1" smd custom (at -0.65 0 90) (size 1 0.5) (layers "B.Cu" "B.Mask")
+    (pad "1" smd custom (at -0.65 0 270) (size 1 0.5) (layers "B.Cu" "B.Mask")
       (net 24 "FOOTSWITCH_1") (pinfunction "A") (pintype "passive") (zone_connect 2) (thermal_bridge_angle 45)
       (options (clearance outline) (anchor rect))
@@
           (width 0) (fill yes))
       ))
-    (pad "2" smd custom (at 0.65 0 90) (size 1 0.5) (layers "B.Cu" "B.Mask")
+    (pad "2" smd custom (at 0.65 0 270) (size 1 0.5) (layers "B.Cu" "B.Mask")
       (net 264 "Net-(JP3-B)") (pinfunction "B") (pintype "passive") (zone_connect 2) (thermal_bridge_angle 45)
       (options (clearance outline) (anchor rect))
@@
   )
   (footprint "Jumper:SolderJumper-2_P1.3mm_Bridged2Bar_RoundedPad1.0x1.5mm" (layer "B.Cu")
-    (at 7 70.35 -90)
-    (descr "SMD Solder Jumper, 1x1.5mm, rounded Pads, 0.3mm gap, bridged with 2 copper strips")
-    (tags "net tie solder jumper bridged")
+    (at 10 73.35 -90)
+    (descr "SMD Solder Jumper, 1x1.5mm, rounded Pads, 0.3mm gap, bridged with 2 copper strips")
+    (tags "net tie solder jumper bridged")

Commit message: fixing ERC stuff, importing PCB into freecad
Parts:
- added D1: 1N5817, Diode_THT:D_DO-41_SOD81_P10.16mm_Horizontal, F.Cu at (7.50, 2.25)
- moved J15 21.1 mm to (19.0, 82.0), turned to 180 degrees
- moved J14 20.1 mm to (35.0, 65.8), turned to 0 degrees
- moved J11 12.4 mm to (2.73, 13.7)
- moved C6 4.85 mm to (22.1, 2.10)
- moved R20 2.12 mm to (42.8, 8.20)
- moved L1 1.66 mm to (24.1, 6.40)
- moved D2 0.54 mm to (16.3, 6.40)
- renumbered D1 to D2, D2 to D3, D3 to D4, D4 to D5, J15 to J14, J16 to J15
Connections:
- C10 pad 1: GNDA -> GND
- C13 pad 1: GNDA -> GND
- C14 pad 2: GNDA -> GND
- C15 pad 2: GNDA -> GND
- C9 pad 1: GNDA -> GND
- D3 pad 1: GNDA -> GND
- D3 pad 2: +3.3VA -> +3.3V
- D4 pad 1: GNDA -> GND
- D4 pad 2: +3.3VA -> +3.3V
- D5 pad 1: Net-(D4-K) -> LED_NEG
- J1 pad 10: LINE_IN_L -> PREAMP_IN_R
- J1 pad 11: LINE_IN_R -> LINE_IN_L
- J1 pad 12: LINE_OUT_L -> LINE_IN_R
- J1 pad 13: LINE_OUT_R -> LINE_OUT_L
- J1 pad 14: LED_NEG -> LINE_OUT_R
- J1 pad 15: GND -> LED_NEG
- J1 pad 3: +3.3V -> +5V
- J1 pad 4: +3.3V -> +5V
- J1 pad 6: JACK_IN -> +3.3V
- J1 pad 7: JACK_OUT -> JACK_IN
- J1 pad 8: PREAMP_IN_L -> JACK_OUT
- J1 pad 9: PREAMP_IN_R -> PREAMP_IN_L
- J11 pad 1: +9V -> GND
- J11 pad 2: GND -> Net-(D1-A)
- J14 pad S: GNDA -> GND
- J14 pad SN: GNDA -> GND
- J14 pad T: Net-(JP11-B) -> JACK_IN
- J14 pad TN: GNDA -> GND
- J15 pad S: GNDA -> GND
- J15 pad SN: GNDA -> GND
- J15 pad T: Net-(JP9-A) -> JACK_OUT
- J15 pad TN: GNDA -> GND
- JP11 pad 2: Net-(JP11-B) -> JACK_IN
- JP4 pad 2: Net-(JP11-B) -> JACK_IN
- JP6 pad 2: GNDA -> GND
- JP7 pad 2: Net-(D4-K) -> LED_NEG
- JP9 pad 1: Net-(JP9-A) -> JACK_OUT
- R4 pad 2: GNDA -> GND
- R5 pad 2: GNDA -> GND
- R7 pad 2: GNDA -> GND
- R9 pad 2: GNDA -> GND
- U1 pad 1: unconnected-(U1-GND-Pad1) -> GND
- U1 pad 15: unconnected-(U1-3V3-Pad15) -> +3.3V
- U1 pad 2: MIDI_IN -> unconnected-(U1-0_RX1_CRX2_CS1-Pad2)
- U1 pad 3: MIDI_OUT -> unconnected-(U1-1_TX1_CTX2_MISO1-Pad3)
- U1 pad 46: unconnected-(U1-3V3-Pad46) -> +3.3V
- U1 pad 47: unconnected-(U1-GND-Pad47) -> GND
- U1 pad 48: unconnected-(U1-VIN-Pad48) -> +5V
- U3 pad 4: GNDA -> GND
Other:
- board text added: "5V"
- board text added: "JACK IN"
- board text added: "JACK OUT"
- board text added: "LINE IN L"
- board text added: "LINE IN R"
- board text added: "LINE OUT L"
- board text added: "LINE OUT R"
- board text added: "P'AMP IN"
- board text added: "P'AMP OUT"

Commit message: save before routing
Parts:
- moved J11 2.37 mm to (5.08, 14.0), turned to -90 degrees
Other:
- board text added: "+"
- board text added: "-"
- board text added: "Bradshaw Instruments Omnistomp V1.0 January 2025"
- board text added: "LED -VE"
- board text added: "PREAMP IN L"

Commit message: <50 unrouted...
Parts:
- moved R14 7.61 mm to (42.3, 34.2), turned to 180 degrees
- moved C14 4.86 mm to (39.1, 30.9)
- moved R16 4.86 mm to (40.8, 30.9)
- moved D3 4.86 mm to (39.8, 24.2)
- moved C19 3.94 mm to (43.3, 14.5)
- moved C20 3.91 mm to (41.5, 14.5)
- moved C22 3.45 mm to (34.2, 14.4)
- moved C16 3.27 mm to (39.1, 27.8), turned to -90 degrees
- moved U5 3.15 mm to (38.3, 12.7)
- moved C24 3.13 mm to (35.1, 11.8)
- moved C23 3.13 mm to (33.2, 11.8)
- moved C18 2.50 mm to (35.6, 6.03)
- moved FB1 2.50 mm to (42.0, 6.10)
- moved U4 2.50 mm to (38.0, 5.66)
- moved C15 2.27 mm to (36.9, 30.9)
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Routing:
- net FOOTSWITCH_6: track 0.00 -> 97.4 mm
- net Net-(U5-LINEOUT_R): track 0.00 -> 80.0 mm
- net Net-(U5-LINEOUT_L): track 0.00 -> 76.9 mm
- net FOOTSWITCH_3: track 0.00 -> 74.9 mm
- net Net-(U3B-+): track 0.00 -> 68.9 mm, vias 0 -> 2
- net LINE_OUT_L: track 0.00 -> 62.2 mm
- net FOOTSWITCH_2: track 0.00 -> 61.6 mm
- net LINE_IN_L: track 0.00 -> 61.3 mm, vias 0 -> 1
- net LINE_IN_R: track 0.00 -> 60.7 mm, vias 0 -> 2
- net LINE_OUT_R: track 0.00 -> 59.7 mm
- net JACK_IN: track 0.00 -> 59.5 mm, vias 0 -> 2
- net +3.3V: track 0.00 -> 51.2 mm, vias 0 -> 3
- net Net-(U3A-+): track 0.00 -> 49.1 mm
- net FOOTSWITCH_9: track 0.00 -> 48.0 mm
- net LED_NEG: track 0.00 -> 46.0 mm
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- added copper zone on B.Cu, net GND

Commit message: 7 unrouted...
Parts:
- moved J12 73.3 mm to (50.8, 12.7), turned to 180 degrees
- moved C22 1.71 mm to (34.0, 16.1)
- moved C24 1.34 mm to (34.5, 13.0)
- moved C23 0.89 mm to (32.8, 12.6)
Routing:
- net PREAMP_IN_L: track 1.62 -> 129.7 mm, vias 0 -> 3
- net PREAMP_IN_R: track 1.62 -> 110.9 mm, vias 0 -> 1
- net +9V: track 35.5 -> 144.1 mm, vias 0 -> 6
- net JACK_OUT: track 0.00 -> 79.5 mm, vias 0 -> 2
- net +3.3V: track 51.2 -> 115.7 mm, vias 3 -> 7
- net JACK_IN: track 59.5 -> 101.0 mm, vias 2 -> 4
- net Net-(J12-Pin_3): track 0.00 -> 37.7 mm, vias 0 -> 2
- net Net-(J12-Pin_1): track 0.00 -> 35.6 mm, vias 0 -> 3
- net Net-(J12-Pin_2): track 0.00 -> 34.6 mm, vias 0 -> 2
- net +5V: track 37.7 -> 69.0 mm, vias 0 -> 1
- net FOOTSWITCH_8: track 11.4 -> 40.6 mm
- net GND: track 42.1 -> 66.3 mm, vias 5 -> 19
- net DAC_SDA: track 25.1 -> 29.2 mm
- net DAC_SCL: track 19.2 -> 22.6 mm
- net Net-(U5-VDDA): track 23.3 -> 26.3 mm
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Other:
- board text added: "P'AMP IN L"
- board text added: "P'AMP IN R"
- board text removed: "P'AMP IN"
- board text removed: "P'AMP OUT"

Commit message: passed ERC!
Parts:
- JP1, JP2, R12, R14: moved to B.Cu
Connections:
- R25 pad 2: +9V -> +3.3V
Routing:
- net +3.3V: track 115.7 -> 181.3 mm
- net GND: track 66.3 -> 112.5 mm, vias 19 -> 22
- net LED_NEG: track 46.0 -> 78.2 mm, vias 0 -> 1
- net PREAMP_IN_L: track 129.7 -> 141.9 mm
- net Net-(JP1-B): track 32.8 -> 40.1 mm
- net FOOTSWITCH_8: track 40.6 -> 46.7 mm, vias 0 -> 1
- net Net-(JP2-A): track 2.23 -> 7.41 mm, vias 0 -> 1
- net LINE_OUT_L: track 62.2 -> 63.4 mm, vias 0 -> 1
- net Net-(JP2-B): track 14.4 -> 15.6 mm
- net Net-(JP1-A): track 2.60 -> 3.59 mm, vias 0 -> 1
- net PREAMP_IN_R: track 110.9 -> 111.5 mm
- net FOOTSWITCH_6: track 97.4 -> 97.9 mm
- net +1V8: vias 1 -> 0
Other:
- board text added: "G"
- board text added: "INPUT"
- board text added: "JACK IN TO PREAMP"
- board text added: "L"
- board text added: "LEFT 4.7K"
- board text added: "OUTPUT"
- board text added: "PHONES"
- board text added: "R"
- board text added: "RIGHT 4.7K"

Commit message: pcb done
Parts:
- L1: footprint Inductor_SMD:L_Changjiang_FNR4020S -> Inductor_SMD:L_Sunlord_SWPA6045S
- moved C2 7.00 mm to (13.0, 9.00)
- moved D2 2.33 mm to (14.0, 6.00)
- moved U2 2.24 mm to (13.0, 13.0)
- moved C4 2.03 mm to (19.0, 15.6)
- moved C5 2.03 mm to (18.0, 13.1)
- moved R1 2.03 mm to (20.2, 13.0)
- moved R2 2.03 mm to (22.7, 13.1)
- moved R3 2.03 mm to (23.5, 15.6)
- moved L1 1.78 mm to (23.0, 7.80)
- moved C1 1.40 mm to (8.78, 8.00)
- moved C3 1.28 mm to (8.00, 14.0)
- moved C6 0.40 mm to (22.1, 2.50)
Routing:
- net Net-(U2-BOOT): track 8.06 -> 2.80 mm
- net Net-(D2-K): track 10.9 -> 14.7 mm
- net Net-(D1-A): track 20.6 -> 22.1 mm
- net Net-(U2-SS): track 2.54 -> 3.22 mm
- net GND: track 112.5 -> 112.9 mm, vias 22 -> 21
