File: pcb/stomp_00/input.kicad_sch (KiCad schematic)
At the start: 26 parts, among them U2 TL072

Commit message: pcb...
Connections:
- net INSTRUMENT_IN_R: now reaches C13.1, R10.1
Changed lines of the file:
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@@
   (junction (at 114.3 90.17) (diameter 0) (color 0 0 0 0)
   )
-  (junction (at 101.6 139.7) (diameter 0) (color 0 0 0 0)
-  )
   (junction (at 133.35 173.99) (diameter 0) (color 0 0 0 0)
-  )
-  (wire (pts (xy 95.25 139.7) (xy 101.6 139.7))
-    (stroke (width 0) (type default))
   )
   (wire (pts (xy 162.56 129.54) (xy 165.1 129.54))
@@
     (stroke (width 0) (type default))
   )
-  (wire (pts (xy 95.25 134.62) (xy 95.25 139.7))
-    (stroke (width 0) (type default))
-  )
   (wire (pts (xy 170.18 106.68) (xy 170.18 110.49))
     (stroke (width 0) (type default))
@@
       (effects (font (size 1.27 1.27)) (justify right) hide)
     )
+  )
+  (global_label "INSTRUMENT_IN_R" (shape input) (at 95.25 132.08 180) (fields_autoplaced)
+    (effects (font (size 1.27 1.27)) (justify right))
+    (property "Intersheetrefs" "${INTERSHEET_REFS}" (at 75.5923 132.08 0)
+      (effects (font (size 1.27 1.27)) (justify right) hide)
+    )

Commit message: changed voltage regulator
Parts:
- R10, R11, R12, R13, R14, R15, R4, R5, R6, R7, R8, R9: footprint (none) -> Resistor_SMD:R_0603_1608Metric
Changed lines of the file:
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@@
       (effects (font (size 1.27 1.27)))
     )
-    (property "Footprint" "" (at 141.224 78.994 90)
+    (property "Footprint" "Resistor_SMD:R_0603_1608Metric" (at 141.224 78.994 90)
       (effects (font (size 1.27 1.27)) hide)
     )
@@
       (effects (font (size 1.27 1.27)))
     )
-    (property "Footprint" "" (at 118.364 59.944 90)
+    (property "Footprint" "Resistor_SMD:R_0603_1608Metric" (at 118.364 59.944 90)
       (effects (font (size 1.27 1.27)) hide)
     )
@@
       (effects (font (size 1.27 1.27)) (justify left))
     )
-    (property "Footprint" "" (at 115.316 136.144 90)
+    (property "Footprint" "Resistor_SMD:R_0603_1608Metric" (at 115.316 136.144 90)
       (effects (font (size 1.27 1.27)) hide)
     )
@@
       (effects (font (size 1.27 1.27)) (justify left))
     )
-    (property "Footprint" "" (at 115.316 78.994 90)
+    (property "Footprint" "Resistor_SMD:R_0603_1608Metric" (at 115.316 78.994 90)
       (effects (font (size 1.27 1.27)) hide)
     )
@@
       (effects (font (size 1.27 1.27)) (justify left))
     )
-    (property "Footprint" "" (at 102.616 86.614 90)
+    (property "Footprint" "Resistor_SMD:R_0603_1608Metric" (at 102.616 86.614 90)
       (effects (font (size 1.27 1.27)) hide)
     )
@@
       (effects (font (size 1.27 1.27)) (justify left))
     )
-    (property "Footprint" "" (at 115.316 128.524 90)
+    (property "Footprint" "Resistor_SMD:R_0603_1608Metric" (at 115.316 128.524 90)
       (effects (font (size 1.27 1.27)) hide)
     )
@@
       (effects (font (size 1.27 1.27)))
     )
-    (property "Footprint" "" (at 118.364 109.474 90)
+    (property "Footprint" "Resistor_SMD:R_0603_1608Metric" (at 118.364 109.474 90)
       (effects (font (size 1.27 1.27)) hide)
     )
@@
       (effects (font (size 1.27 1.27)))
     )
-    (property "Footprint" "" (at 131.064 68.834 90)
+    (property "Footprint" "Resistor_SMD:R_0603_1608Metric" (at 131.064 68.834 90)
       (effects (font (size 1.27 1.27)) hide)
     )
@@
       (effects (font (size 1.27 1.27)) (justify left))
     )
-    (property "Footprint" "" (at 102.616 136.144 90)
+    (property "Footprint" "Resistor_SMD:R_0603_1608Metric" (at 102.616 136.144 90)
       (effects (font (size 1.27 1.27)) hide)
     )
@@
       (effects (font (size 1.27 1.27)))
     )
-    (property "Footprint" "" (at 131.064 118.364 90)
+    (property "Footprint" "Resistor_SMD:R_0603_1608Metric" (at 131.064 118.364 90)
       (effects (font (size 1.27 1.27)) hide)
     )
@@
       (effects (font (size 1.27 1.27)) (justify left))
     )
-    (property "Footprint" "" (at 115.316 86.614 90)
+    (property "Footprint" "Resistor_SMD:R_0603_1608Metric" (at 115.316 86.614 90)
       (effects (font (size 1.27 1.27)) hide)
     )
@@
       (effects (font (size 1.27 1.27)))
     )
-    (property "Footprint" "" (at 141.224 128.524 90)
-      (effects (font (size 1.27 1.27)) hide)
-    )
+    (property "Footprint" "Resistor_SMD:R_0603_1608Metric" (at 141.224 128.524 90)
+      (effects (font (size 1.27 1.27)) hide)
+    )

Commit message: tidying up dac connections
Parts:
- C10, C11, C12, C13, C14, C15, C16, C17, C18, C7, C8: footprint (none) -> Capacitor_SMD:C_0603_1608Metric
Changed lines of the file:
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@@
       (effects (font (size 1.27 1.27)))
     )
-    (property "Footprint" "" (at 134.62 109.5248 0)
+    (property "Footprint" "Capacitor_SMD:C_0603_1608Metric" (at 134.62 109.5248 0)
       (effects (font (size 1.27 1.27)) hide)
     )
@@
       (effects (font (size 1.27 1.27)))
     )
-    (property "Footprint" "" (at 114.3 109.5248 0)
+    (property "Footprint" "Capacitor_SMD:C_0603_1608Metric" (at 114.3 109.5248 0)
       (effects (font (size 1.27 1.27)) hide)
     )
@@
       (effects (font (size 1.27 1.27)))
     )
-    (property "Footprint" "" (at 152.4 130.5052 0)
+    (property "Footprint" "Capacitor_SMD:C_0603_1608Metric" (at 152.4 130.5052 0)
       (effects (font (size 1.27 1.27)) hide)
     )
@@
       (effects (font (size 1.27 1.27)) (justify left))
     )
-    (property "Footprint" "" (at 147.0152 137.16 0)
+    (property "Footprint" "Capacitor_SMD:C_0603_1608Metric" (at 147.0152 137.16 0)
       (effects (font (size 1.27 1.27)) hide)
     )
@@
       (effects (font (size 1.27 1.27)) (justify left))
     )
-    (property "Footprint" "" (at 147.0152 87.63 0)
+    (property "Footprint" "Capacitor_SMD:C_0603_1608Metric" (at 147.0152 87.63 0)
       (effects (font (size 1.27 1.27)) hide)
     )
@@
       (effects (font (size 1.27 1.27)))
     )
-    (property "Footprint" "" (at 152.4 80.9752 0)
+    (property "Footprint" "Capacitor_SMD:C_0603_1608Metric" (at 152.4 80.9752 0)
       (effects (font (size 1.27 1.27)) hide)
     )
@@
       (effects (font (size 1.27 1.27)))
     )
-    (property "Footprint" "" (at 111.76 131.1148 0)
+    (property "Footprint" "Capacitor_SMD:C_0603_1608Metric" (at 111.76 131.1148 0)
       (effects (font (size 1.27 1.27)) hide)
     )
@@
       (effects (font (size 1.27 1.27)))
     )
-    (property "Footprint" "" (at 111.76 81.5848 0)
+    (property "Footprint" "Capacitor_SMD:C_0603_1608Metric" (at 111.76 81.5848 0)
       (effects (font (size 1.27 1.27)) hide)
     )
@@
       (effects (font (size 1.27 1.27)))
     )
-    (property "Footprint" "" (at 134.62 59.9948 0)
+    (property "Footprint" "Capacitor_SMD:C_0603_1608Metric" (at 134.62 59.9948 0)
       (effects (font (size 1.27 1.27)) hide)
     )
@@
       (effects (font (size 1.27 1.27)))
     )
-    (property "Footprint" "" (at 114.3 59.9948 0)
+    (property "Footprint" "Capacitor_SMD:C_0603_1608Metric" (at 114.3 59.9948 0)
       (effects (font (size 1.27 1.27)) hide)
     )
@@
       (effects (font (size 1.27 1.27)) (justify right))
     )
-    (property "Footprint" "" (at 143.8148 162.56 0)
-      (effects (font (size 1.27 1.27)) hide)
-    )
+    (property "Footprint" "Capacitor_SMD:C_0603_1608Metric" (at 143.8148 162.56 0)
+      (effects (font (size 1.27 1.27)) hide)
+    )

Commit message: not much
Parts:
- renumbered C14 to C10, C10 to C11, C15 to C12, C18 to C13, C12 to C14, C16 to C15, C11 to C16, C8 to C7, C13 to C8, C7 to C9, D1 to D2, D4 to D3, R5 to R10, R13 to R11, R8 to R12, R14 to R13, R9 to R14, R10 to R5, R11 to R8, R12 to R9

Commit message: layout getting closer
Parts:
- added JP1, JP2: Jumper_2_Bridged, Jumper:SolderJumper-2_P1.3mm_Bridged2Bar_RoundedPad1.0x1.5mm, symbol Jumper:Jumper_2_Bridged
- added R12, R14: Gain, Resistor_THT:R_Axial_DIN0207_L6.3mm_D2.5mm_P7.62mm_Horizontal, symbol Device:R_US
- R13: renamed from R12; value 4.2k -> 4.7k
- R15: renamed from R13; value 4.2k -> 4.7k
- renumbered R14 to R16, R15 to R17
Connections:
- net at C12.1, R11.2, R15.1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: now also R14.1
- net at C12.2, R17.1, U2.7: now also JP2.2 (B), R14.2; no longer R15.2
- net at C11.2, R16.1, U2.1: now also JP1.2 (B), R12.2; no longer R13.2
- net at C11.1, R10.2, R13.1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: now also R12.1
- net INSTRUMENT_IN_L renamed PREAMP_IN_L
- net INSTRUMENT_IN_R renamed PREAMP_IN_R
- new net: JP2.1 (A), R15.2
- new net: JP1.1 (A), R13.2
Other:
- moved on the sheet: C11, C14, C15, C16, C17, C8, C9, D2, D3, R10, R15, R16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

Commit message: fixing ERC stuff, importing PCB into freecad
Parts:
- renumbered D2 to D3, D3 to D4
Connections:
- net +3.3VA renamed +3.3V
- net GNDA renamed GND
