File: pcb/stomp_00/power.kicad_sch (KiCad schematic)
At the start: 13 parts, among them J11 Barrel_Jack, U2 TPS54331DR

Commit message: fixing ERC stuff, importing PCB into freecad
Parts:
- added D1: 1N5817, Diode_THT:D_DO-41_SOD81_P10.16mm_Horizontal, symbol Diode:1N5817
- renumbered D1 to D2
Connections:
- net +9V: now also D1.1 (K); no longer J11.1
- net GND: now also J11.1; no longer J11.2
- new net: D1.2 (A), J11.2
Other:
- moved on the sheet: J11
Changed lines of the file:
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@@
   (junction (at 185.42 85.09) (diameter 0) (color 0 0 0 0)
   )
+  (junction (at 74.93 57.15) (diameter 0) (color 0 0 0 0)
+  )
   (junction (at 161.29 118.11) (diameter 0) (color 0 0 0 0)
   )
@@
   )
   (no_connect (at 119.38 100.33))
+  (wire (pts (xy 64.77 62.23) (xy 78.74 62.23))
+    (stroke (width 0) (type default))
+  )
   (wire (pts (xy 177.8 124.46) (xy 177.8 102.87))
     (stroke (width 0) (type default))
@@
     (stroke (width 0) (type default))
   )
-  (wire (pts (xy 73.66 57.15) (xy 80.01 57.15))
+  (wire (pts (xy 72.39 57.15) (xy 74.93 57.15))
     (stroke (width 0) (type default))
   )
@@
     (stroke (width 0) (type default))
   )
-  (wire (pts (xy 80.01 62.23) (xy 80.01 65.405))
+  (wire (pts (xy 78.74 62.23) (xy 78.74 66.04))
     (stroke (width 0) (type default))
   )
@@
     (stroke (width 0) (type default))
   )
-  (wire (pts (xy 73.66 62.23) (xy 80.01 62.23))
-    (stroke (width 0) (type default))
-  )
   (wire (pts (xy 177.8 102.87) (xy 185.42 102.87))
     (stroke (width 0) (type default))
@@
     (stroke (width 0) (type default))
   )
-  (wire (pts (xy 80.01 57.15) (xy 80.01 54.61))
+  (wire (pts (xy 78.74 57.15) (xy 78.74 54.61))
     (stroke (width 0) (type default))
   )
@@
     (stroke (width 0) (type default))
   )
+  (wire (pts (xy 74.93 48.26) (xy 74.93 57.15))
+    (stroke (width 0) (type default))
+  )
   (wire (pts (xy 119.38 95.25) (xy 113.03 95.25))
+    (stroke (width 0) (type default))
+  )
+  (wire (pts (xy 74.93 57.15) (xy 78.74 57.15))
     (stroke (width 0) (type default))
   )
@@
     (fill (type none))
     (effects (font (size 1.27 1.27)) (justify left top))
+  )
+  (symbol (lib_id "power:PWR_FLAG") (at 74.93 48.26 0) (unit 1)
+    (in_bom yes) (on_board yes) (dnp no) (fields_autoplaced)
+    (property "Reference" "#FLG03" (at 74.93 46.355 0)
+      (effects (font (size 1.27 1.27)) hide)
+    )
+    (property "Value" "PWR_FLAG" (at 74.93 44.7581 0)
+      (effects (font (size 1.27 1.27)))
+    )
+    (property "Footprint" "" (at 74.93 48.26 0)
+      (effects (font (size 1.27 1.27)) hide)
+    )
+    (property "Datasheet" "~" (at 74.93 48.26 0)
+      (effects (font (size 1.27 1.27)) hide)
+    )
+    (pin "1")
+    (instances
+      (project "stomp_00"
+        (path "/8f4a2eb0-078b-46cb-b534-a4acd11d130e/72df8ca6-692f-47f3-a8bd-ce94f6cd776a"
+          (reference "#FLG03") (unit 1)
+        )
+      )
+    )
   )
   (symbol (lib_id "Device:R_US") (at 185.42 106.68 0) (unit 1)
@@
         )
         (path "/8f4a2eb0-078b-46cb-b534-a4acd11d130e/72df8ca6-692f-47f3-a8bd-ce94f6cd776a"
-          (reference "#PWR08") (unit 1)
+          (reference "#PWR014") (unit 1)
         )
         (path "/8f4a2eb0-078b-46cb-b534-a4acd11d130e/9942492d-ba8b-45b2-b427-7fe14bedb7e0"
@@
     )
   )
-  (symbol (lib_id "Connector:Barrel_Jack") (at 66.04 59.69 0) (unit 1)
-    (in_bom yes) (on_board yes) (dnp no) (fields_autoplaced)
-    (property "Reference" "J11" (at 66.04 52.8701 0)
-      (effects (font (size 1.27 1.27)))
-    )
-    (property "Value" "Barrel_Jack" (at 66.04 54.7911 0)
-      (effects (font (size 1.27 1.27)))
-    )
-    (property "Footprint" "Connector_PinHeader_2.54mm:PinHeader_1x02_P2.54mm_Vertical" (at 67.31 60.706 0)
-      (effects (font (size 1.27 1.27)) hide)
-    )
-    (property "Datasheet" "~" (at 67.31 60.706 0)
+  (symbol (lib_id "Connector:Barrel_Jack") (at 57.15 59.69 0) (mirror x) (unit 1)
+    (in_bom yes) (on_board yes) (dnp no)
+    (property "Reference" "J11" (at 57.15 66.5099 0)
+      (effects (font (size 1.27 1.27)))
+    )
+    (property "Value" "Barrel_Jack" (at 57.15 64.5889 0)
+      (effects (font (size 1.27 1.27)))
+    )
+    (property "Footprint" "Connector_PinHeader_2.54mm:PinHeader_1x02_P2.54mm_Vertical" (at 58.42 58.674 0)
+      (effects (font (size 1.27 1.27)) hide)
+    )
+    (property "Datasheet" "~" (at 58.42 58.674 0)
       (effects (font (size 1.27 1.27)) hide)
     )
@@
         )
         (path "/8f4a2eb0-078b-46cb-b534-a4acd11d130e/72df8ca6-692f-47f3-a8bd-ce94f6cd776a"
-          (reference "#PWR07") (unit 1)
+          (reference "#PWR013") (unit 1)
         )
         (path "/8f4a2eb0-078b-46cb-b534-a4acd11d130e/9942492d-ba8b-45b2-b427-7fe14bedb7e0"
@@
     )
   )
-  (symbol (lib_id "power:GND") (at 80.01 65.405 0) (unit 1)
-    (in_bom yes) (on_board yes) (dnp no) (fields_autoplaced)
-    (property "Reference" "#PWR068" (at 80.01 71.755 0)
-      (effects (font (size 1.27 1.27)) hide)
-    )
-    (property "Value" "GND" (at 80.01 69.5405 0)
-      (effects (font (size 1.27 1.27)))
-    )
-    (property "Footprint" "" (at 80.01 65.405 0)
-      (effects (font (size 1.27 1.27)) hide)
-    )
-    (property "Datasheet" "" (at 80.01 65.405 0)
+  (symbol (lib_id "power:GND") (at 78.74 66.04 0) (unit 1)
+    (in_bom yes) (on_board yes) (dnp no) (fields_autoplaced)
+    (property "Reference" "#PWR068" (at 78.74 72.39 0)
+      (effects (font (size 1.27 1.27)) hide)
+    )
+    (property "Value" "GND" (at 78.74 70.1755 0)
+      (effects (font (size 1.27 1.27)))
+    )
+    (property "Footprint" "" (at 78.74 66.04 0)
+      (effects (font (size 1.27 1.27)) hide)
+    )
+    (property "Datasheet" "" (at 78.74 66.04 0)
       (effects (font (size 1.27 1.27)) hide)
     )
@@
         )
         (path "/8f4a2eb0-078b-46cb-b534-a4acd11d130e/72df8ca6-692f-47f3-a8bd-ce94f6cd776a"
-          (reference "#PWR05") (unit 1)
+          (reference "#PWR011") (unit 1)
         )
         (path "/8f4a2eb0-078b-46cb-b534-a4acd11d130e/9942492d-ba8b-45b2-b427-7fe14bedb7e0"
@@
     )
   )
+  (symbol (lib_id "Diode:1N5817") (at 68.58 57.15 0) (mirror y) (unit 1)
+    (in_bom yes) (on_board yes) (dnp no)
+    (property "Reference" "D1" (at 68.8975 52.8701 0)
+      (effects (font (size 1.27 1.27)))
+    )
+    (property "Value" "1N5817" (at 68.8975 54.7911 0)
+      (effects (font (size 1.27 1.27)))
+    )
+    (property "Footprint" "Diode_THT:D_DO-41_SOD81_P10.16mm_Horizontal" (at 68.58 61.595 0)
+      (effects (font (size 1.27 1.27)) hide)
+    )
+    (property "Datasheet" "http://www.vishay.com/docs/88525/1n5817.pdf" (at 68.58 57.15 0)
+      (effects (font (size 1.27 1.27)) hide)
+    )
+    (pin "1")
+    (pin "2")
+    (instances
+      (project "stomp_00"
+        (path "/8f4a2eb0-078b-46cb-b534-a4acd11d130e/72df8ca6-692f-47f3-a8bd-ce94f6cd776a"
+          (reference "D1") (unit 1)
+        )
+      )
+    )
+  )
   (symbol (lib_id "Device:C") (at 114.3 107.95 0) (unit 1)
     (in_bom yes) (on_board yes) (dnp no) (fields_autoplaced)
@@
     )
   )
-  (symbol (lib_id "power:+9V") (at 80.01 54.61 0) (unit 1)
-    (in_bom yes) (on_board yes) (dnp no) (fields_autoplaced)
-    (property "Reference" "#PWR07" (at 80.01 58.42 0)
-      (effects (font (size 1.27 1.27)) hide)
-    )
-    (property "Value" "+9V" (at 80.01 51.1081 0)
-      (effects (font (size 1.27 1.27)))
-    )
-    (property "Footprint" "" (at 80.01 54.61 0)
-      (effects (font (size 1.27 1.27)) hide)
-    )
-    (property "Datasheet" "" (at 80.01 54.61 0)
+  (symbol (lib_id "power:+9V") (at 78.74 54.61 0) (unit 1)
+    (in_bom yes) (on_board yes) (dnp no) (fields_autoplaced)
+    (property "Reference" "#PWR07" (at 78.74 58.42 0)
+      (effects (font (size 1.27 1.27)) hide)
+    )
+    (property "Value" "+9V" (at 78.74 51.1081 0)
+      (effects (font (size 1.27 1.27)))
+    )
+    (property "Footprint" "" (at 78.74 54.61 0)
+      (effects (font (size 1.27 1.27)) hide)
+    )
+    (property "Datasheet" "" (at 78.74 54.61 0)
       (effects (font (size 1.27 1.27)) hide)
     )
@@
         )
         (path "/8f4a2eb0-078b-46cb-b534-a4acd11d130e/72df8ca6-692f-47f3-a8bd-ce94f6cd776a"
-          (reference "#PWR04") (unit 1)
+          (reference "#PWR010") (unit 1)
         )
         (path "/8f4a2eb0-078b-46cb-b534-a4acd11d130e/9942492d-ba8b-45b2-b427-7fe14bedb7e0"
@@
         )
         (path "/8f4a2eb0-078b-46cb-b534-a4acd11d130e/72df8ca6-692f-47f3-a8bd-ce94f6cd776a"
-          (reference "#PWR09") (unit 1)
+          (reference "#PWR015") (unit 1)
         )
         (path "/8f4a2eb0-078b-46cb-b534-a4acd11d130e/9942492d-ba8b-45b2-b427-7fe14bedb7e0"
@@
         )
         (path "/8f4a2eb0-078b-46cb-b534-a4acd11d130e/72df8ca6-692f-47f3-a8bd-ce94f6cd776a"
-          (reference "#PWR010") (unit 1)
+          (reference "#PWR016") (unit 1)
         )
         (path "/8f4a2eb0-078b-46cb-b534-a4acd11d130e/9942492d-ba8b-45b2-b427-7fe14bedb7e0"
@@
   (symbol (lib_id "Diode:B340") (at 151.13 91.44 270) (unit 1)
     (in_bom yes) (on_board yes) (dnp no) (fields_autoplaced)
-    (property "Reference" "D1" (at 153.162 90.4788 90)
+    (property "Reference" "D2" (at 153.162 90.4788 90)
       (effects (font (size 1.27 1.27)) (justify left))
     )
@@
       (project "stomp_00"
         (path "/8f4a2eb0-078b-46cb-b534-a4acd11d130e/72df8ca6-692f-47f3-a8bd-ce94f6cd776a"
-          (reference "D1") (unit 1)
+          (reference "D2") (unit 1)
         )
       )
@@
         )
         (path "/8f4a2eb0-078b-46cb-b534-a4acd11d130e/72df8ca6-692f-47f3-a8bd-ce94f6cd776a"
-          (reference "#PWR06") (unit 1)
+          (reference "#PWR012") (unit 1)
         )
         (path "/8f4a2eb0-078b-46cb-b534-a4acd11d130e/9942492d-ba8b-45b2-b427-7fe14bedb7e0"
