File: pcb/stomp_00/power.kicad_sch (KiCad schematic)
At the start: 14 parts, among them J11 Barrel_Jack, U2 TPS54331DR

Commit message: pcb done
Parts:
- L1: footprint Inductor_SMD:L_Changjiang_FNR4020S -> Inductor_SMD:L_Sunlord_SWPA6045S
Changed lines of the file:
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@@
       (effects (font (size 1.27 1.27)))
     )
-    (property "Footprint" "Inductor_SMD:L_Changjiang_FNR4020S" (at 158.75 85.09 0)
+    (property "Footprint" "Inductor_SMD:L_Sunlord_SWPA6045S" (at 158.75 85.09 0)
       (effects (font (size 1.27 1.27)) hide)
     )
