File: pcb/stomp_00/dac.kicad_sch (KiCad schematic)
At the start: 20 parts, among them J1 Headphones, U11 AP7313-18SAG, U3 SGTL5000XNLA3

Commit message: not much
Parts:
- renumbered C2 to C18, C3 to C19, C4 to C20, C1 to C21, C25 to C22, C5 to C23, C9 to C24, C21 to C25, C22 to C26, J1 to J12, R2 to R16, R1 to R17, R3 to R18, R17 to R19, R18 to R20, R19 to R21, R20 to R22, U3 to U5

Commit message: layout getting closer
Parts:
- renumbered R16 to R18, R17 to R19, R18 to R20, R19 to R21, R20 to R22, R21 to R23, R22 to R24
Changed lines of the file:
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@@
   (symbol (lib_id "Device:R_US") (at 180.34 95.25 180) (unit 1)
     (in_bom yes) (on_board yes) (dnp no) (fields_autoplaced)
-    (property "Reference" "R19" (at 181.991 94.6063 0)
+    (property "Reference" "R21" (at 181.991 94.6063 0)
       (effects (font (size 1.27 1.27)) (justify right))
     )
@@
       (project "stomp_00"
         (path "/8f4a2eb0-078b-46cb-b534-a4acd11d130e/7598c0f0-0137-4b50-80b5-b929d25c284a"
-          (reference "R19") (unit 1)
+          (reference "R21") (unit 1)
         )
       )
@@
   (symbol (lib_id "Device:R_US") (at 111.76 96.52 270) (unit 1)
     (in_bom yes) (on_board yes) (dnp no) (fields_autoplaced)
-    (property "Reference" "R18" (at 111.76 92.6211 90)
+    (property "Reference" "R20" (at 111.76 92.6211 90)
       (effects (font (size 1.27 1.27)))
     )
@@
       (project "stomp_00"
         (path "/8f4a2eb0-078b-46cb-b534-a4acd11d130e/7598c0f0-0137-4b50-80b5-b929d25c284a"
-          (reference "R18") (unit 1)
+          (reference "R20") (unit 1)
         )
       )
@@
   (symbol (lib_id "Device:R_US") (at 189.23 95.25 180) (unit 1)
     (in_bom yes) (on_board yes) (dnp no) (fields_autoplaced)
-    (property "Reference" "R20" (at 190.881 94.6063 0)
+    (property "Reference" "R22" (at 190.881 94.6063 0)
       (effects (font (size 1.27 1.27)) (justify right))
     )
@@
       (project "stomp_00"
         (path "/8f4a2eb0-078b-46cb-b534-a4acd11d130e/7598c0f0-0137-4b50-80b5-b929d25c284a"
-          (reference "R20") (unit 1)
+          (reference "R22") (unit 1)
         )
       )
@@
   (symbol (lib_id "Device:R_US") (at 107.95 109.22 180) (unit 1)
     (in_bom yes) (on_board yes) (dnp no) (fields_autoplaced)
-    (property "Reference" "R17" (at 109.601 108.5763 0)
+    (property "Reference" "R19" (at 109.601 108.5763 0)
       (effects (font (size 1.27 1.27)) (justify right))
     )
@@
       (project "stomp_00"
         (path "/8f4a2eb0-078b-46cb-b534-a4acd11d130e/7598c0f0-0137-4b50-80b5-b929d25c284a"
-          (reference "R17") (unit 1)
+          (reference "R19") (unit 1)
         )
       )
@@
   (symbol (lib_id "Device:R_US") (at 99.06 109.22 180) (unit 1)
     (in_bom yes) (on_board yes) (dnp no) (fields_autoplaced)
-    (property "Reference" "R16" (at 100.711 108.5763 0)
+    (property "Reference" "R18" (at 100.711 108.5763 0)
       (effects (font (size 1.27 1.27)) (justify right))
     )
@@
       (project "stomp_00"
         (path "/8f4a2eb0-078b-46cb-b534-a4acd11d130e/7598c0f0-0137-4b50-80b5-b929d25c284a"
-          (reference "R16") (unit 1)
+          (reference "R18") (unit 1)
         )
       )
@@
   (symbol (lib_id "Device:R_US") (at 201.93 88.9 270) (unit 1)
     (in_bom yes) (on_board yes) (dnp no) (fields_autoplaced)
-    (property "Reference" "R22" (at 201.93 85.0011 90)
+    (property "Reference" "R24" (at 201.93 85.0011 90)
       (effects (font (size 1.27 1.27)))
     )
@@
       (project "stomp_00"
         (path "/8f4a2eb0-078b-46cb-b534-a4acd11d130e/7598c0f0-0137-4b50-80b5-b929d25c284a"
-          (reference "R22") (unit 1)
+          (reference "R24") (unit 1)
         )
       )
@@
   (symbol (lib_id "Device:R_US") (at 201.93 81.28 270) (unit 1)
     (in_bom yes) (on_board yes) (dnp no) (fields_autoplaced)
-    (property "Reference" "R21" (at 201.93 77.3811 90)
+    (property "Reference" "R23" (at 201.93 77.3811 90)
       (effects (font (size 1.27 1.27)))
     )
@@
       (project "stomp_00"
         (path "/8f4a2eb0-078b-46cb-b534-a4acd11d130e/7598c0f0-0137-4b50-80b5-b929d25c284a"
-          (reference "R21") (unit 1)
-        )
-      )
+          (reference "R23") (unit 1)
+        )
+      )

Commit message: fixing ERC stuff, importing PCB into freecad
Changed lines of the file:
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@@
 (kicad_sch (version 20230121) (generator eeschema)
   (paper "A4")
+  (junction (at 152.4 49.53) (diameter 0) (color 0 0 0 0)
+  )
   (junction (at 85.09 49.53) (diameter 0) (color 0 0 0 0)
   )
@@
     (stroke (width 0) (type default))
   )
-  (wire (pts (xy 148.59 49.53) (xy 156.21 49.53))
+  (wire (pts (xy 148.59 49.53) (xy 152.4 49.53))
     (stroke (width 0) (type default))
   )
@@
   )
   (wire (pts (xy 185.42 99.06) (xy 189.23 99.06))
+    (stroke (width 0) (type default))
+  )
+  (wire (pts (xy 152.4 49.53) (xy 156.21 49.53))
     (stroke (width 0) (type default))
   )
@@
         )
         (path "/8f4a2eb0-078b-46cb-b534-a4acd11d130e/7598c0f0-0137-4b50-80b5-b929d25c284a"
-          (reference "#PWR030") (unit 1)
+          (reference "#PWR036") (unit 1)
+        )
+      )
+    )
+  )
+  (symbol (lib_id "power:PWR_FLAG") (at 152.4 49.53 0) (unit 1)
+    (in_bom yes) (on_board yes) (dnp no) (fields_autoplaced)
+    (property "Reference" "#FLG04" (at 152.4 47.625 0)
+      (effects (font (size 1.27 1.27)) hide)
+    )
+    (property "Value" "PWR_FLAG" (at 152.4 46.0281 0)
+      (effects (font (size 1.27 1.27)))
+    )
+    (property "Footprint" "" (at 152.4 49.53 0)
+      (effects (font (size 1.27 1.27)) hide)
+    )
+    (property "Datasheet" "~" (at 152.4 49.53 0)
+      (effects (font (size 1.27 1.27)) hide)
+    )
+    (pin "1")
+    (instances
+      (project "stomp_00"
+        (path "/8f4a2eb0-078b-46cb-b534-a4acd11d130e/7598c0f0-0137-4b50-80b5-b929d25c284a"
+          (reference "#FLG04") (unit 1)
         )
       )
@@
         )
         (path "/8f4a2eb0-078b-46cb-b534-a4acd11d130e/7598c0f0-0137-4b50-80b5-b929d25c284a"
-          (reference "#PWR032") (unit 1)
+          (reference "#PWR038") (unit 1)
         )
       )
@@
         )
         (path "/8f4a2eb0-078b-46cb-b534-a4acd11d130e/7598c0f0-0137-4b50-80b5-b929d25c284a"
-          (reference "#PWR031") (unit 1)
+          (reference "#PWR037") (unit 1)
         )
       )
@@
         )
         (path "/8f4a2eb0-078b-46cb-b534-a4acd11d130e/7598c0f0-0137-4b50-80b5-b929d25c284a"
-          (reference "#PWR028") (unit 1)
+          (reference "#PWR034") (unit 1)
         )
       )
@@
   (symbol (lib_id "power:+3.3V") (at 104.14 105.41 0) (unit 1)
     (in_bom yes) (on_board yes) (dnp no) (fields_autoplaced)
-    (property "Reference" "#PWR026" (at 104.14 109.22 0)
+    (property "Reference" "#PWR032" (at 104.14 109.22 0)
       (effects (font (size 1.27 1.27)) hide)
     )
@@
       (project "stomp_00"
         (path "/8f4a2eb0-078b-46cb-b534-a4acd11d130e/7598c0f0-0137-4b50-80b5-b929d25c284a"
-          (reference "#PWR026") (unit 1)
+          (reference "#PWR032") (unit 1)
         )
       )
@@
         )
         (path "/8f4a2eb0-078b-46cb-b534-a4acd11d130e/7598c0f0-0137-4b50-80b5-b929d25c284a"
-          (reference "#PWR029") (unit 1)
+          (reference "#PWR035") (unit 1)
         )
       )
@@
         )
         (path "/8f4a2eb0-078b-46cb-b534-a4acd11d130e/7598c0f0-0137-4b50-80b5-b929d25c284a"
-          (reference "#PWR027") (unit 1)
+          (reference "#PWR033") (unit 1)
         )
       )
@@
         )
         (path "/8f4a2eb0-078b-46cb-b534-a4acd11d130e/7598c0f0-0137-4b50-80b5-b929d25c284a"
-          (reference "#PWR025") (unit 1)
-        )
-      )
+          (reference "#PWR031") (unit 1)
+        )
+      )
