File: pcb/stomp_00/footswitch.kicad_sch (KiCad schematic)
At the start: 16 parts, among them J2 GuitarInput1, J2 GuitarOutput1, J5 Conn_01x09, J6 Conn_01x09, SW2 Footswitch

Commit message: tweaking layout, issue with usb socket placement
Parts:
- J2: footprint Connector_Audio:Jack_6.35mm_Neutrik_NMJ4HCD2_Horizontal -> stomp:Jack_6.35mm_Neutrik_NMJ4HCD2_Horizontal
Changed lines of the file:
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@@
       (effects (font (size 1.27 1.27)))
     )
-    (property "Footprint" "Connector_Audio:Jack_6.35mm_Neutrik_NMJ4HCD2_Horizontal" (at 212.09 69.85 0)
+    (property "Footprint" "stomp:Jack_6.35mm_Neutrik_NMJ4HCD2_Horizontal" (at 212.09 69.85 0)
       (effects (font (size 1.27 1.27)) hide)
     )
@@
       (effects (font (size 1.27 1.27)))
     )
-    (property "Footprint" "Connector_Audio:Jack_6.35mm_Neutrik_NMJ4HCD2_Horizontal" (at 212.09 100.33 0)
-      (effects (font (size 1.27 1.27)) hide)
-    )
+    (property "Footprint" "stomp:Jack_6.35mm_Neutrik_NMJ4HCD2_Horizontal" (at 212.09 100.33 0)
+      (effects (font (size 1.27 1.27)) hide)
+    )

Commit message: tidying up footprints, layout, etc
Parts:
- removed J6: Conn_01x09, Connector_PinHeader_2.54mm:PinHeader_1x09_P2.54mm_Vertical, symbol Connector_Generic:Conn_01x09
- added J6: Conn_02x05_Counter_Clockwise, Connector_PinHeader_2.54mm:PinHeader_2x05_P2.54mm_Vertical, symbol Connector_Generic:Conn_02x05_Counter_Clockwise
- J5: footprint Connector_PinHeader_2.54mm:PinHeader_1x09_P2.54mm_Vertical -> stomp:PinHeader_3x03_P2.54mm_Vertical_footswitch_breakout
Changed lines of the file:
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@@
+    )
+  )
+  (symbol (lib_id "Connector_Generic:Conn_02x05_Counter_Clockwise") (at 149.86 39.37 0) (unit 1)
+    (in_bom yes) (on_board yes) (dnp no) (fields_autoplaced)
+    (property "Reference" "J6" (at 151.13 30.0101 0)
+      (effects (font (size 1.27 1.27)))
+    )
+    (property "Value" "Conn_02x05_Counter_Clockwise" (at 151.13 31.9311 0)
+      (effects (font (size 1.27 1.27)))
+    )
+    (property "Footprint" "Connector_PinHeader_2.54mm:PinHeader_2x05_P2.54mm_Vertical" (at 149.86 39.37 0)
+      (effects (font (size 1.27 1.27)) hide)
+    )
+    (property "Datasheet" "~" (at 149.86 39.37 0)
+      (effects (font (size 1.27 1.27)) hide)
+    )
+    (pin "1")
+    (pin "10")
+    (pin "2")
+    (pin "3")
+    (pin "4")
+    (pin "5")
+    (pin "6")
+    (pin "7")
+    (pin "8")
+    (pin "9")
+    (instances
+      (project "stomp_00"
+        (path "/8f4a2eb0-078b-46cb-b534-a4acd11d130e/8515bfbc-58f4-43ce-a6da-807641c93feb"
+          (reference "J6") (unit 1)
+        )
+      )
     )
   )
@@
       (effects (font (size 1.27 1.27)))
     )
-    (property "Footprint" "Connector_PinHeader_2.54mm:PinHeader_1x09_P2.54mm_Vertical" (at 101.6 48.26 0)
+    (property "Footprint" "stomp:PinHeader_3x03_P2.54mm_Vertical_footswitch_breakout" (at 101.6 48.26 0)
       (effects (font (size 1.27 1.27)) hide)
     )
@@
         )
       )
-    )
-  )
-  (symbol (lib_id "Connector_Generic:Conn_01x09") (at 153.67 48.26 90) (unit 1)
-    (in_bom yes) (on_board yes) (dnp no) (fields_autoplaced)
-    (property "Reference" "J6" (at 153.67 43.9801 90)
-      (effects (font (size 1.27 1.27)))
-    )
-    (property "Value" "Conn_01x09" (at 153.67 45.9011 90)
-      (effects (font (size 1.27 1.27)))
-    )
-    (property "Footprint" "Connector_PinHeader_2.54mm:PinHeader_1x09_P2.54mm_Vertical" (at 153.67 48.26 0)
-      (effects (font (size 1.27 1.27)) hide)
-    )
-    (property "Datasheet" "~" (at 153.67 48.26 0)
-      (effects (font (size 1.27 1.27)) hide)
-    )
-    (pin "1")
-    (pin "2")
-    (pin "3")
-    (pin "4")
-    (pin "5")
-    (pin "6")
-    (pin "7")
-    (pin "8")
-    (pin "9")
-    (instances
-      (project "stomp_00"
-        (path "/8f4a2eb0-078b-46cb-b534-a4acd11d130e"
-          (reference "J6") (unit 1)
-        )
-        (path "/8f4a2eb0-078b-46cb-b534-a4acd11d130e/8515bfbc-58f4-43ce-a6da-807641c93feb"
-          (reference "J6") (unit 1)
-        )
-      )

Commit message: tidying up dac connections
Parts:
- J5: value Conn_01x09 -> Footswitch_breakout
Changed lines of the file:
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@@
       (effects (font (size 1.27 1.27)))
     )
-    (property "Value" "Conn_01x09" (at 101.6 45.9011 90)
+    (property "Value" "Footswitch_breakout" (at 101.6 45.9011 90)
       (effects (font (size 1.27 1.27)))
     )

Commit message: not much
Parts:
- renumbered J6 to J14
Changed lines of the file:
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@@
         )
         (path "/8f4a2eb0-078b-46cb-b534-a4acd11d130e/8515bfbc-58f4-43ce-a6da-807641c93feb"
-          (reference "J3") (unit 1)
+          (reference "J15") (unit 1)
         )
       )
@@
         )
         (path "/8f4a2eb0-078b-46cb-b534-a4acd11d130e/8515bfbc-58f4-43ce-a6da-807641c93feb"
-          (reference "D5") (unit 1)
+          (reference "D4") (unit 1)
         )
       )
@@
   (symbol (lib_id "Connector_Generic:Conn_02x05_Counter_Clockwise") (at 149.86 39.37 0) (unit 1)
     (in_bom yes) (on_board yes) (dnp no) (fields_autoplaced)
-    (property "Reference" "J6" (at 151.13 30.0101 0)
+    (property "Reference" "J14" (at 151.13 30.0101 0)
       (effects (font (size 1.27 1.27)))
     )
@@
       (project "stomp_00"
         (path "/8f4a2eb0-078b-46cb-b534-a4acd11d130e/8515bfbc-58f4-43ce-a6da-807641c93feb"
-          (reference "J6") (unit 1)
+          (reference "J14") (unit 1)
         )
       )
@@
         )
         (path "/8f4a2eb0-078b-46cb-b534-a4acd11d130e/8515bfbc-58f4-43ce-a6da-807641c93feb"
-          (reference "SW2") (unit 2)
+          (reference "SW1") (unit 2)
         )
       )
@@
         )
         (path "/8f4a2eb0-078b-46cb-b534-a4acd11d130e/8515bfbc-58f4-43ce-a6da-807641c93feb"
-          (reference "R16") (unit 1)
+          (reference "R23") (unit 1)
         )
       )
@@
         )
         (path "/8f4a2eb0-078b-46cb-b534-a4acd11d130e/8515bfbc-58f4-43ce-a6da-807641c93feb"
-          (reference "SW2") (unit 1)
+          (reference "SW1") (unit 1)
         )
       )
@@
         )
         (path "/8f4a2eb0-078b-46cb-b534-a4acd11d130e/8515bfbc-58f4-43ce-a6da-807641c93feb"
-          (reference "J2") (unit 1)
+          (reference "J13") (unit 1)
         )
       )
@@
         )
         (path "/8f4a2eb0-078b-46cb-b534-a4acd11d130e/8515bfbc-58f4-43ce-a6da-807641c93feb"
-          (reference "J5") (unit 1)
+          (reference "J16") (unit 1)
         )
       )
@@
         )
         (path "/8f4a2eb0-078b-46cb-b534-a4acd11d130e/8515bfbc-58f4-43ce-a6da-807641c93feb"
-          (reference "SW2") (unit 3)
-        )
-      )
+          (reference "SW1") (unit 3)
+        )
+      )

Commit message: layout getting closer
Parts:
- removed J14: Conn_02x05_Counter_Clockwise, Connector_PinHeader_2.54mm:PinHeader_2x05_P2.54mm_Vertical, symbol Connector_Generic:Conn_02x05_Counter_Clockwise
- renumbered JP9 to JP11
Connections:
- net JACK_IN: now reaches J2.T, JP11.2 (B), JP3.2 (B)
- net LED_NEG: now reaches D5.1 (K), JP6.2 (B)
- net JACK_OUT: now reaches J2.T, JP8.1 (A)
- net INSTRUMENT_IN_L renamed PREAMP_IN_L
Other:
- moved on the sheet: D5, J2, JP11, R16

Commit message: fixing ERC stuff, importing PCB into freecad
Connections:
- net GNDA renamed GND
Changed lines of the file:
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@@
     (stroke (width 0) (type default))
-  )
-  (text_box "Breakout pins for:\ninput jack (open jumper to circuit in)\noutput jack (open jumper from circuit out)\ncircuit in L\ncircuit in R\ncircuit out L\ncircuit out R\nheadphone out L/R?\nled negative?"
-    (at 203.2 7.62 0) (size 52.07 25.4)
-    (stroke (width 0) (type default))
-    (fill (type none))
-    (effects (font (size 1.27 1.27)) (justify left top))
-  )
-  (text_box "Add default routing with cuttable traces:\n\n1: 7\n2: guitar input tip\n3: circuit audio input\n\n4: not connected\n5: ground\n6: led negative\n\n7: 1\n8: guitar output tip\n9: circuit audio output"
-    (at 20.32 15.24 0) (size 43.18 30.48)
-    (stroke (width 0) (type default))
-    (fill (type none))
-    (effects (font (size 1.27 1.27)) (justify left top))
   )
   (global_label "FOOTSWITCH_9" (shape output) (at 46.99 88.9 0) (fields_autoplaced)
@@
         )
         (path "/8f4a2eb0-078b-46cb-b534-a4acd11d130e/8515bfbc-58f4-43ce-a6da-807641c93feb"
-          (reference "J15") (unit 1)
+          (reference "J14") (unit 1)
         )
       )
@@
         )
         (path "/8f4a2eb0-078b-46cb-b534-a4acd11d130e/8515bfbc-58f4-43ce-a6da-807641c93feb"
-          (reference "D4") (unit 1)
+          (reference "D5") (unit 1)
         )
       )
@@
         )
         (path "/8f4a2eb0-078b-46cb-b534-a4acd11d130e/8515bfbc-58f4-43ce-a6da-807641c93feb"
-          (reference "J16") (unit 1)
-        )
-      )
-    )
-  )
-  (symbol (lib_id "power:GNDA") (at 184.15 104.14 0) (unit 1)
+          (reference "J15") (unit 1)
+        )
+      )
+    )
+  )
+  (symbol (lib_id "power:GND") (at 184.15 104.14 0) (unit 1)
     (in_bom yes) (on_board yes) (dnp no) (fields_autoplaced)
     (property "Reference" "#PWR033" (at 184.15 110.49 0)
       (effects (font (size 1.27 1.27)) hide)
     )
-    (property "Value" "GNDA" (at 184.15 108.2755 0)
+    (property "Value" "GND" (at 184.15 107.95 0)
       (effects (font (size 1.27 1.27)))
     )
@@
         )
         (path "/8f4a2eb0-078b-46cb-b534-a4acd11d130e/8515bfbc-58f4-43ce-a6da-807641c93feb"
-          (reference "#PWR033") (unit 1)
+          (reference "#PWR039") (unit 1)
         )
       )
@@
         )
         (path "/8f4a2eb0-078b-46cb-b534-a4acd11d130e/8515bfbc-58f4-43ce-a6da-807641c93feb"
-          (reference "#PWR034") (unit 1)
-        )
-      )
+          (reference "#PWR040") (unit 1)
+        )
+      )

Commit message: passed ERC!
Connections:
- net +9V renamed +3.3V
Changed lines of the file:
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@@
     )
   )
-  (symbol (lib_id "power:+9V") (at 204.47 83.82 0) (unit 1)
+  (symbol (lib_id "power:+3.3V") (at 204.47 83.82 0) (unit 1)
     (in_bom yes) (on_board yes) (dnp no) (fields_autoplaced)
-    (property "Reference" "#PWR034" (at 204.47 87.63 0)
+    (property "Reference" "#PWR?" (at 204.47 87.63 0)
       (effects (font (size 1.27 1.27)) hide)
     )
-    (property "Value" "+9V" (at 204.47 80.3181 0)
+    (property "Value" "+3.3V" (at 204.47 80.264 0)
       (effects (font (size 1.27 1.27)))
     )
@@
     (instances
       (project "stomp_00"
+        (path "/8f4a2eb0-078b-46cb-b534-a4acd11d130e/9942492d-ba8b-45b2-b427-7fe14bedb7e0"
+          (reference "#PWR?") (unit 1)
+        )
         (path "/8f4a2eb0-078b-46cb-b534-a4acd11d130e"
-          (reference "#PWR034") (unit 1)
+          (reference "#PWR08") (unit 1)
         )
         (path "/8f4a2eb0-078b-46cb-b534-a4acd11d130e/8515bfbc-58f4-43ce-a6da-807641c93feb"
