File: pcb/stomp_01/footswitch.kicad_sch (KiCad schematic)
At the start: 15 parts, among them J2 GuitarInput1, J2 GuitarOutput1, J5 Footswitch_breakout, SW2 Footswitch

Commit message: looking nice
Parts:
- removed J2: GuitarInput1, stomp:Jack_6.35mm_Neutrik_NMJ4HCD2_Horizontal, symbol Connector_Audio:NMJ4HCD2
- removed J2: GuitarOutput1, stomp:Jack_6.35mm_Neutrik_NMJ4HCD2_Horizontal, symbol Connector_Audio:NMJ4HCD2
- added J14: GuitarInput1, Connector_Wire:SolderWire-1sqmm_1x02_P5.4mm_D1.4mm_OD2.7mm, symbol Connector_Generic:Conn_01x02
- added J15: GuitarOutput1, Connector_Wire:SolderWire-1sqmm_1x02_P5.4mm_D1.4mm_OD2.7mm, symbol Connector_Generic:Conn_01x02
- renumbered J5 to J13, JP9 to JP10, JP1 to JP3, JP3 to JP4, JP4 to JP5, JP2 to JP6, JP6 to JP7, JP7 to JP8, JP8 to JP9, R16 to R25, SW2 to SW1
Connections:
- net GND: now also J14.2 (Pin_2), J15.2 (Pin_2)
- net JACK_IN: now also J14.1 (Pin_1)
- net JACK_OUT: now also J15.1 (Pin_1)
