File: pcb/stomp_01/stomp_01.kicad_sch (KiCad schematic)
At the start: 13 parts, among them J1 Conn_01x18_Pin, J10 Conn_01x18_Pin, J2 Conn_01x18_Pin, J3 Conn_01x18_Pin, J4 Conn_01x18_Pin, J5 Conn_01x18_Pin, J6 Conn_01x18_Pin, J7 Conn_01x18_Pin, J8 Conn_01x18_Pin, J9 Conn_01x18_Pin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

Commit message: looking nice
Parts:
- removed J2, J5, J6, J7, J9: Conn_01x18_Pin, stomp:PinHeader_1x18_P2.54mm_Vertical_perf, symbol Connector:Conn_01x18_Pin
- added H3, H4: MountingHole, MountingHole:MountingHole_3.2mm_M3, symbol Mechanical:MountingHole
- added J10: Conn_01x18_Pin, stomp:PinHeader_1x18_P2.54mm_Vertical_perf, symbol Connector:Conn_01x18_Pin
- added J4, J5, J6, J7: Conn_01x18_Pin, stomp:PinHeader_1x24_P2.54mm_Vertical_perf, symbol Connector:Conn_01x24_Pin
- renumbered J3 to J2, J4 to J3, J10 to J9
Connections:
- no-connect marks 198 -> 222

Commit message: pre routing
Connections:
- net HEADPHONES_LEFT: now reaches J4.1 (Pin_1)
- net HEADPHONES_GND: now reaches J4.2 (Pin_2)
- net HEADPHONES_RIGHT: now reaches J4.3 (Pin_3)
- no-connect marks 222 -> 219
Other:
- moved on the sheet: J10, J5, J6, J7, J8, J9
