File: pcb/stomp_01/stomp_01.kicad_pcb (KiCad board)
At the start: 2 copper layers, 54 x 104 mm, 92 parts, among them J1 Conn_01x18_Pin, J10 Conn_01x18_Pin, J11 Barrel_Jack, J12 Headphones, J13 Footswitch_breakout, J14 GuitarInput1, J15 GuitarOutput1, J2 Conn_01x18_Pin, J3 Conn_01x18_Pin, J4 Conn_01x18_Pin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

Commit message: more tweaks
Parts:
- moved J1 173.1 mm to (-158.3, 74.8)
- moved J2 173.1 mm to (-155.8, 74.8)
- moved J3 173.1 mm to (-153.2, 74.8)
- moved J4 173.1 mm to (-150.7, 74.8)
- moved J5 173.1 mm to (-148.2, 74.8)
- moved J6 173.1 mm to (-145.6, 74.8)
- moved J7 173.1 mm to (-143.1, 74.8)
- moved J8 173.1 mm to (-140.5, 74.8)
- moved J9 173.1 mm to (-138.0, 74.8)
- moved C14 116.3 mm to (-77.2, 29.2)
- moved C15 116.3 mm to (-79.5, 29.2)
- moved C16 116.3 mm to (-77.2, 26.1)
- moved C17 116.3 mm to (-79.5, 26.1)
- moved C22 116.3 mm to (-82.3, 14.4)
- moved JP2 116.3 mm to (-79.7, 35.9)
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
Commit message: looking nice
Parts:
- removed the J2 at (-155.8, 74.8)
- removed the J9 at (-138.0, 74.8)
- added H3: MountingHole, MountingHole:MountingHole_3.2mm_M3, F.Cu at (83.0, 134.0)
- added H4: MountingHole, MountingHole:MountingHole_3.2mm_M3, F.Cu at (127.0, 134.0)
- added J10: Conn_01x18_Pin, stomp:PinHeader_1x18_P2.54mm_Vertical_perf, F.Cu at (127.5, 64.0)
- added J4: Conn_01x18_Pin, stomp:PinHeader_1x24_P2.54mm_Vertical_perf, F.Cu at (89.4, 48.8)
- J14, J15: footprint stomp:Jack_6.35mm_Neutrik_NMJ4HCD2_Horizontal -> Connector_Wire:SolderWire-1sqmm_1x02_P5.4mm_D1.4mm_OD2.7mm
- J5, J6, J7: footprint stomp:PinHeader_1x18_P2.54mm_Vertical_perf -> stomp:PinHeader_1x24_P2.54mm_Vertical_perf
- moved J6 264.3 mm to (117.4, 48.8)
- moved J7 264.3 mm to (119.9, 48.8)
- moved J8 263.2 mm to (122.5, 64.0)
- moved J5 241.5 mm to (92.0, 48.8)
- moved J1 240.4 mm to (81.8, 64.0)
- moved J2 237.8 mm to (84.3, 64.0)
- moved J3 237.8 mm to (86.9, 64.0)
- moved J12 211.2 mm to (154.0, 64.1)
- moved C14 188.3 mm to (105.5, 75.0)
- moved C15 188.3 mm to (103.2, 75.0)
- moved C16 188.3 mm to (105.5, 72.0)
- moved C17 188.3 mm to (103.2, 72.0)
- moved C22 188.3 mm to (100.3, 60.3)
- moved JP2 188.3 mm to (102.9, 81.8)
- moved R10 188.3 mm to (108.2, 93.3)
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- renumbered J3 to J2, J4 to J3, J10 to J9
Other:
- board text added: "Above PCB shape should fit 1590B, metal or polycarbonate. 104 x 54 with 8mm corner cutouts, rounded to 5mm radius. Keepouts added to prevent components/copper touching enclosure."
- board text removed: "Above PCB shape should fit 1590B, metal or polycarbonate. 104 x 54 with 8mm corner cutouts, rounded to 5mm radius."

Commit message: pre routing
Parts:
- removed J12: Headphones, Connector_PinHeader_2.54mm:PinHeader_1x03_P2.54mm_Vertical
- J11: footprint Connector_PinHeader_2.54mm:PinHeader_1x02_P2.54mm_Vertical -> Connector_Wire:SolderWire-1sqmm_1x02_P5.4mm_D1.4mm_OD2.7mm
- moved R22 37.9 mm to (84.0, 122.0)
- moved C25 37.9 mm to (84.0, 119.0)
- moved R23 37.9 mm to (84.0, 125.2)
- moved R21 37.9 mm to (82.4, 122.0)
- moved C26 37.9 mm to (82.4, 119.0)
- moved R24 37.9 mm to (82.4, 125.2)
- moved R5 35.9 mm to (92.0, 124.8)
- moved R4 35.9 mm to (88.9, 124.8)
- moved C7 35.9 mm to (88.9, 123.2)
- moved C8 35.9 mm to (92.0, 123.2)
- moved R6 35.9 mm to (88.9, 120.0)
- moved R7 35.9 mm to (92.0, 120.0)
- moved R8 35.9 mm to (88.9, 121.6)
- moved R9 35.9 mm to (92.0, 121.6)
- moved JP11 6.35 mm to (127.3, 116.8)
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Connections:
- J4 pad 1: unconnected-(J4-Pin_1-Pad1) -> HEADPHONES_LEFT
- J4 pad 2: unconnected-(J4-Pin_2-Pad2) -> HEADPHONES_GND
- J4 pad 3: unconnected-(J4-Pin_3-Pad3) -> HEADPHONES_RIGHT
- U5 pad 1: Net-(J12-Pin_1) -> HEADPHONES_RIGHT
- U5 pad 2: Net-(J12-Pin_2) -> HEADPHONES_GND
- U5 pad 4: Net-(J12-Pin_3) -> HEADPHONES_LEFT
Other:
- board text added: "Bradshaw Instruments Omnistomp V1.01 May 2025"
- board text removed: "Bradshaw Instruments Omnistomp V1.0 January 2025"

Commit message: 100 unrouted
Parts:
- moved C21 1.02 mm to (104.3, 52.8)
- moved C18 1.00 mm to (101.7, 50.2)
- moved FB1 1.00 mm to (107.9, 49.2)
- moved R20 1.00 mm to (107.9, 51.0)
- moved U4 1.00 mm to (104.4, 50.0)
- moved C3 0.75 mm to (101.5, 113.3)
- moved C24 0.61 mm to (101.4, 57.1)
- moved C23 0.45 mm to (99.5, 56.6)
Routing:
- net Net-(U5-LINEOUT_R): track 0.00 -> 77.5 mm
- net Net-(U5-LINEOUT_L): track 0.00 -> 73.7 mm
- net Net-(U3A-+): track 0.00 -> 46.9 mm
- net Net-(U3B-+): track 0.00 -> 43.7 mm, vias 0 -> 2
- net DAC_DOUT: track 0.00 -> 32.2 mm, vias 0 -> 1
- net +3.3V: track 0.00 -> 32.1 mm
- net GND: track 0.00 -> 31.1 mm, vias 0 -> 3
- net DAC_DIN: track 0.00 -> 26.5 mm, vias 0 -> 1
- net DAC_SDA: track 0.00 -> 24.8 mm, vias 0 -> 2
- net HEADPHONES_LEFT: track 0.00 -> 24.8 mm
- net DAC_SCL: track 0.00 -> 23.8 mm, vias 0 -> 2
- net HEADPHONES_RIGHT: track 0.00 -> 21.1 mm
- net HEADPHONES_GND: track 0.00 -> 15.7 mm
- net Net-(JP2-B): track 0.00 -> 15.6 mm
- net DAC_LRCLK: track 0.00 -> 15.2 mm
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- added copper zone on In1.Cu, net GND
Other:
- copper layers 2 -> 4

Commit message: 53 unrouted
Routing:
- net JACK_IN: track 0.00 -> 123.1 mm, vias 0 -> 2
- net PREAMP_IN_L: track 0.00 -> 103.4 mm, vias 0 -> 3
- net +9V: track 2.24 -> 85.0 mm
- net LINE_OUT_L: track 0.00 -> 66.4 mm, vias 0 -> 2
- net +5V: track 2.54 -> 54.9 mm
- net FOOTSWITCH_8: track 0.00 -> 43.2 mm
- net FOOTSWITCH_2: track 0.00 -> 39.3 mm
- net FOOTSWITCH_9: track 0.00 -> 34.2 mm, vias 0 -> 1
- net FOOTSWITCH_7: track 0.00 -> 34.0 mm
- net FOOTSWITCH_3: track 0.00 -> 32.0 mm, vias 0 -> 1
- net FOOTSWITCH_6: track 0.00 -> 31.4 mm
- net FOOTSWITCH_5: track 0.00 -> 30.9 mm, vias 0 -> 1
- net LED_NEG: track 0.00 -> 30.2 mm, vias 0 -> 1
- net FOOTSWITCH_1: track 0.00 -> 29.0 mm
- net JACK_OUT: track 0.00 -> 21.4 mm
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- added copper zone on In2.Cu, net +3.3V

Commit message: zero unrouted
Routing:
- net +9V: track 85.0 -> 212.0 mm, vias 0 -> 3
- net +5V: track 54.9 -> 149.6 mm, vias 0 -> 1
- net LINE_OUT_R: track 0.00 -> 52.8 mm, vias 0 -> 5
- net PREAMP_IN_R: track 1.62 -> 53.8 mm, vias 0 -> 2
- net JACK_OUT: track 21.4 -> 67.4 mm, vias 0 -> 1
- net LINE_IN_L: track 13.6 -> 56.2 mm, vias 0 -> 1
- net LINE_IN_R: track 14.1 -> 56.0 mm, vias 0 -> 1
- net GND: track 32.7 -> 71.7 mm, vias 3 -> 19
- net LED_NEG: track 30.2 -> 54.5 mm, vias 1 -> 2
- net Net-(U5-VDDA): track 2.48 -> 18.1 mm, vias 0 -> 2
- net Net-(D2-K): track 0.00 -> 12.7 mm
- net Net-(U2-VSENSE): track 0.00 -> 9.82 mm
- net Net-(U2-COMP): track 0.00 -> 5.55 mm
- net Net-(C25-Pad2): track 0.00 -> 5.21 mm
- net +3.3V: track 34.6 -> 39.6 mm, vias 0 -> 4
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